Commit message: update to new urdf, get assert_surface_types to work

File: knowledge/urdf/hsrb_lab.urdf (robot description, URDF)
Before this commit: robot hsrb_lab, 24 links, 23 joints
Links:
- added link shelf_small_back_piece; collision box size=0.01 0.71 1.04; visual box size=0.01 0.71 1.04
- added link shelf_small_base_center
- added link shelf_small_center
- added link shelf_small_door_left_door; collision box size=0.01 0.355 1.04; visual box size=0.01 0.355 1.04
- added link shelf_small_floor_0_piece; collision box size=0.34 0.71 0.02; visual box size=0.34 0.71 0.02
- added link shelf_small_floor_1_piece; collision box size=0.34 0.71 0.015; visual box size=0.34 0.71 0.015
- added link shelf_small_floor_2_piece; collision box size=0.34 0.71 0.015; visual box size=0.34 0.71 0.015
- added link shelf_small_floor_3_piece; collision box size=0.34 0.71 0.02; visual box size=0.34 0.71 0.02
- added link shelf_small_left_side_piece; collision box size=0.34 0.01 1.04; visual box size=0.34 0.01 1.04
- added link shelf_small_origin
- added link shelf_small_right_side_piece; collision box size=0.34 0.01 1.04; visual box size=0.34 0.01 1.04
- added link table_2_center; collision box size=0.55 0.95 0.72; visual box size=0.55 0.95 0.72
- added link table_2_front_edge_center
- added link table_2_origin
- added link table_2_surface_center
- added link table_3_center; collision box size=0.55 0.55 0.45; visual box size=0.55 0.55 0.45
- added link table_3_front_edge_center
- added link table_3_origin
- added link table_3_surface_center
Joints:
- added joint shelf_small_back_piece_joint: type fixed, parent shelf_small_origin, child shelf_small_back_piece, origin xyz=0.34 0.355 0.52 rpy=0 0 0
- added joint shelf_small_base_center_joint: type fixed, parent shelf_small_origin, child shelf_small_base_center, origin xyz=0.17 0.355 0.0 rpy=0 0 0
- added joint shelf_small_center_joint: type fixed, parent shelf_small_origin, child shelf_small_center, origin xyz=0.17 0.355 0.52 rpy=0 0 0
- added joint shelf_small_door_left_door_joint: type revolute, parent shelf_small_left_side_piece, child shelf_small_door_left_door, origin xyz=-0.17 -0.1775 0 rpy=0 0 3.1416, axis 0 0 1, limit lower=0.0 upper=1.91986 effort=30 velocity=1.0
- added joint shelf_small_floor_0_piece_joint: type fixed, parent shelf_small_base_center, child shelf_small_floor_0_piece, origin xyz=0.0 0.0 0.055 rpy=0 0 0
- added joint shelf_small_floor_1_piece_joint: type fixed, parent shelf_small_base_center, child shelf_small_floor_1_piece, origin xyz=0.0 0.0 0.45 rpy=0 0 0
- added joint shelf_small_floor_2_piece_joint: type fixed, parent shelf_small_base_center, child shelf_small_floor_2_piece, origin xyz=0.0 0.0 0.71 rpy=0 0 0
- added joint shelf_small_floor_3_piece_joint: type fixed, parent shelf_small_base_center, child shelf_small_floor_3_piece, origin xyz=0.0 0.0 1.02 rpy=0 0 0
- added joint shelf_small_left_side_piece_joint: type fixed, parent shelf_small_origin, child shelf_small_left_side_piece, origin xyz=0.17 0.71 0.52 rpy=0 0 0
- added joint shelf_small_origin_joint: type fixed, parent room_link, child shelf_small_origin, origin xyz=-0.95 -0.1 0 rpy=0 0 -1.570796327
- added joint shelf_small_right_side_piece_joint: type fixed, parent shelf_small_origin, child shelf_small_right_side_piece, origin xyz=0.17 0.0 0.52 rpy=0 0 0
- added joint table_2_center_joint: type fixed, parent table_2_origin, child table_2_center, origin xyz=0.275 0.475 0.36 rpy=0 0 0
- added joint table_2_front_edge_center_joint: type fixed, parent table_2_origin, child table_2_front_edge_center, origin xyz=0 0.475 0.72 rpy=0 0 0
- added joint table_2_origin_joint: type fixed, parent room_link, child table_2_origin, origin xyz=-1.7025 1.2 0 rpy=0 0 3.14159265359
- added joint table_2_surface_center_joint: type fixed, parent table_2_origin, child table_2_surface_center, origin xyz=0.275 0.475 0.72 rpy=0 0 0
- added joint table_3_center_joint: type fixed, parent table_3_origin, child table_3_center, origin xyz=0.275 0.275 0.225 rpy=0 0 0
- added joint table_3_front_edge_center_joint: type fixed, parent table_3_origin, child table_3_front_edge_center, origin xyz=0 0.275 0.45 rpy=0 0 0
- added joint table_3_origin_joint: type fixed, parent room_link, child table_3_origin, origin xyz=2.3 1 0 rpy=0 0 3.14159265359
- added joint table_3_surface_center_joint: type fixed, parent table_3_origin, child table_3_surface_center, origin xyz=0.275 0.275 0.45 rpy=0 0 0
- joint shelf_origin_joint: origin xyz=-0.1 -0.3 0 rpy=0 0 -1.570796327 -> xyz=0.0 -0.1 0 rpy=0 0 -1.570796327
- joint table_area_2_main_joint: origin xyz=-0.35 2.15 0 rpy=0 0 3.14159265359 -> xyz=0.25 2.35 0 rpy=0 0 3.14159265359
- joint table_area_main_joint: origin xyz=1.85 2.15 0 rpy=0 0 3.14159265359 -> xyz=2.35 2.35 0 rpy=0 0 3.14159265359
- joint table_origin_joint: origin xyz=-3 0 0 rpy=0 0 -1.655 -> xyz=-2.5 0.2 0 rpy=0 0 -1.655
- joint walls_main_joint: origin xyz=-0.5 1 0 rpy=0 0 0 -> xyz=0 1.2 0 rpy=0 0 0

Commit message: udate urdf AGAIN!

File: knowledge/urdf/hsrb_lab.urdf (robot description, URDF)
Before this commit: robot hsrb_lab, 28 links, 27 joints
Links:
- added link shelf_small_back_piece; collision box size=0.01 0.71 1.04; visual box size=0.01 0.71 1.04
- added link shelf_small_base_center
- added link shelf_small_center
- added link shelf_small_door_left_door; collision box size=0.01 0.355 1.04; visual box size=0.01 0.355 1.04
- added link shelf_small_floor_0_piece; collision box size=0.34 0.71 0.02; visual box size=0.34 0.71 0.02
- added link shelf_small_floor_1_piece; collision box size=0.34 0.71 0.015; visual box size=0.34 0.71 0.015
- added link shelf_small_floor_2_piece; collision box size=0.34 0.71 0.015; visual box size=0.34 0.71 0.015
- added link shelf_small_floor_3_piece; collision box size=0.34 0.71 0.02; visual box size=0.34 0.71 0.02
- added link shelf_small_left_side_piece; collision box size=0.34 0.01 1.04; visual box size=0.34 0.01 1.04
- added link shelf_small_origin
- added link shelf_small_right_side_piece; collision box size=0.34 0.01 1.04; visual box size=0.34 0.01 1.04
- added link table_3_center; collision box size=0.55 0.55 0.45; visual box size=0.55 0.55 0.45
- added link table_3_front_edge_center
- added link table_3_origin
- added link table_3_surface_center
Joints:
- added joint shelf_small_back_piece_joint: type fixed, parent shelf_small_origin, child shelf_small_back_piece, origin xyz=0.34 0.355 0.52 rpy=0 0 0
- added joint shelf_small_base_center_joint: type fixed, parent shelf_small_origin, child shelf_small_base_center, origin xyz=0.17 0.355 0.0 rpy=0 0 0
- added joint shelf_small_center_joint: type fixed, parent shelf_small_origin, child shelf_small_center, origin xyz=0.17 0.355 0.52 rpy=0 0 0
- added joint shelf_small_door_left_door_joint: type revolute, parent shelf_small_left_side_piece, child shelf_small_door_left_door, origin xyz=-0.17 -0.1775 0 rpy=0 0 3.1416, axis 0 0 1, limit lower=0.0 upper=1.91986 effort=30 velocity=1.0
- added joint shelf_small_floor_0_piece_joint: type fixed, parent shelf_small_base_center, child shelf_small_floor_0_piece, origin xyz=0.0 0.0 0.055 rpy=0 0 0
- added joint shelf_small_floor_1_piece_joint: type fixed, parent shelf_small_base_center, child shelf_small_floor_1_piece, origin xyz=0.0 0.0 0.45 rpy=0 0 0
- added joint shelf_small_floor_2_piece_joint: type fixed, parent shelf_small_base_center, child shelf_small_floor_2_piece, origin xyz=0.0 0.0 0.71 rpy=0 0 0
- added joint shelf_small_floor_3_piece_joint: type fixed, parent shelf_small_base_center, child shelf_small_floor_3_piece, origin xyz=0.0 0.0 1.02 rpy=0 0 0
- added joint shelf_small_left_side_piece_joint: type fixed, parent shelf_small_origin, child shelf_small_left_side_piece, origin xyz=0.17 0.71 0.52 rpy=0 0 0
- added joint shelf_small_origin_joint: type fixed, parent room_link, child shelf_small_origin, origin xyz=-0.95 -0.1 0 rpy=0 0 -1.570796327
- added joint shelf_small_right_side_piece_joint: type fixed, parent shelf_small_origin, child shelf_small_right_side_piece, origin xyz=0.17 0.0 0.52 rpy=0 0 0
- added joint table_3_center_joint: type fixed, parent table_3_origin, child table_3_center, origin xyz=0.275 0.275 0.225 rpy=0 0 0
- added joint table_3_front_edge_center_joint: type fixed, parent table_3_origin, child table_3_front_edge_center, origin xyz=0 0.275 0.45 rpy=0 0 0
- added joint table_3_origin_joint: type fixed, parent room_link, child table_3_origin, origin xyz=2.3 1 0 rpy=0 0 3.14159265359
- added joint table_3_surface_center_joint: type fixed, parent table_3_origin, child table_3_surface_center, origin xyz=0.275 0.275 0.45 rpy=0 0 0
- joint shelf_origin_joint: origin xyz=-0.1 -0.3 0 rpy=0 0 -1.570796327 -> xyz=0.0 -0.1 0 rpy=0 0 -1.570796327
- joint table_area_2_main_joint: origin xyz=-0.35 2.15 0 rpy=0 0 3.14159265359 -> xyz=0.25 2.35 0 rpy=0 0 3.14159265359
- joint table_area_main_joint: origin xyz=1.85 2.15 0 rpy=0 0 3.14159265359 -> xyz=2.35 2.35 0 rpy=0 0 3.14159265359
- joint table_origin_joint: origin xyz=-3 0 0 rpy=0 0 -1.655 -> xyz=-2.5 0.2 0 rpy=0 0 -1.655
- joint walls_main_joint: origin xyz=-0.5 1 0 rpy=0 0 0 -> xyz=0 1.2 0 rpy=0 0 0

Commit message: update urdf to fit map

File: knowledge/urdf/hsrb_lab.urdf (robot description, URDF)
Before this commit: robot hsrb_lab, 43 links, 42 joints
Joints:
- joint world_room_joint: origin xyz=0.0 0.0 0  rpy=0 0 0 -> xyz=0.0 0.12 0  rpy=0 0 0

Commit message: update urdf for new map

File: knowledge/urdf/hsrb_lab.urdf (robot description, URDF)
Before this commit: robot hsrb_lab, 43 links, 42 joints
Joints:
- joint shelf_origin_joint: origin xyz=0.0 -0.1 0 rpy=0 0 -1.570796327 -> xyz=0.1 -0.1 0 rpy=0 0 -1.570796327
- joint world_room_joint: origin xyz=0.0 0.12 0  rpy=0 0 0 -> xyz=0.0 0 0  rpy=0 0 0

Commit message: update  urdf

File: knowledge/urdf/hsrb_lab.urdf (robot description, URDF)
Before this commit: robot hsrb_lab, 43 links, 42 joints
Joints:
- joint world_room_joint: origin xyz=0.0 0 0  rpy=0 0 0 -> xyz=0.0 0.12 0  rpy=0 0 0
