Commit message: rotate T1

File: knowledge/urdf/robocup_sim_t1.urdf (robot description, URDF)
Before this commit: robot hsrb_lab, 34 links, 33 joints
Joints:
- joint table_origin_joint: origin xyz=-0.25 1.7 0 rpy=0 0 2.35619449019 -> xyz=-0.25 1.7 0 rpy=0 0 3.141

Commit message: fix

File: knowledge/urdf/robocup_sim_t1.urdf (robot description, URDF)
Before this commit: robot hsrb_lab, 34 links, 33 joints
Joints:
- joint table_origin_joint: origin xyz=-0.25 1.7 0 rpy=0 0 3.141 -> xyz=-0.21 1.66 0 rpy=0 0 1.5707
