Commit message: extended test environment

File: knowledge/urdf/gz_sim_v1_openable_door.urdf (robot description, URDF)
Before this commit: robot hsrb_lab, 40 links, 39 joints
Links:
- removed link bed_table_center
- removed link bed_table_front_edge_center
- removed link bed_table_origin
- removed link bed_table_surface_center
- removed link hcr_shefl_2_back_piece
- removed link hcr_shefl_2_base_center
- removed link hcr_shefl_2_center
- removed link hcr_shefl_2_floor_0_piece
- removed link hcr_shefl_2_floor_1_piece
- removed link hcr_shefl_2_floor_2_piece
- removed link hcr_shefl_2_left_side_piece
- removed link hcr_shefl_2_origin
- removed link hcr_shefl_2_right_side_piece
- added link bookshelf_clone_back_piece; collision box size=0.01 0.88 0.9; visual box size=0.01 0.88 0.9
- added link bookshelf_clone_base_center
- added link bookshelf_clone_center
- added link bookshelf_clone_floor_0_piece; collision box size=0.4 0.88 0.04; visual box size=0.4 0.88 0.04
- added link bookshelf_clone_floor_1_piece; collision box size=0.4 0.88 0.04; visual box size=0.4 0.88 0.04
- added link bookshelf_clone_floor_2_piece; collision box size=0.4 0.88 0.04; visual box size=0.4 0.88 0.04
- added link bookshelf_clone_left_side_piece; collision box size=0.4 0.01 0.9; visual box size=0.4 0.01 0.9
- added link bookshelf_clone_origin
- added link bookshelf_clone_right_side_piece; collision box size=0.4 0.01 0.9; visual box size=0.4 0.01 0.9
Joints:
- removed joint bed_table_center_joint
- removed joint bed_table_front_edge_center_joint
- removed joint bed_table_origin_joint
- removed joint bed_table_surface_center_joint
- removed joint hcr_shefl_2_back_piece_joint
- removed joint hcr_shefl_2_base_center_joint
- removed joint hcr_shefl_2_center_joint
- removed joint hcr_shefl_2_floor_0_piece_joint
- removed joint hcr_shefl_2_floor_1_piece_joint
- removed joint hcr_shefl_2_floor_2_piece_joint
- removed joint hcr_shefl_2_left_side_piece_joint
- removed joint hcr_shefl_2_origin_joint
- removed joint hcr_shefl_2_right_side_piece_joint
- added joint bookshelf_clone_back_piece_joint: type fixed, parent bookshelf_clone_origin, child bookshelf_clone_back_piece, origin xyz=0.4 0.44 0.45 rpy=0 0 0
- added joint bookshelf_clone_base_center_joint: type fixed, parent bookshelf_clone_origin, child bookshelf_clone_base_center, origin xyz=0.2 0.44 0.0 rpy=0 0 0
- added joint bookshelf_clone_center_joint: type fixed, parent bookshelf_clone_origin, child bookshelf_clone_center, origin xyz=0.2 0.44 0.45 rpy=0 0 0
- added joint bookshelf_clone_floor_0_piece_joint: type fixed, parent bookshelf_clone_base_center, child bookshelf_clone_floor_0_piece, origin xyz=0.0 0.0 0.06 rpy=0 0 0
- added joint bookshelf_clone_floor_1_piece_joint: type fixed, parent bookshelf_clone_base_center, child bookshelf_clone_floor_1_piece, origin xyz=0.0 0.0 0.44 rpy=0 0 0
- added joint bookshelf_clone_floor_2_piece_joint: type fixed, parent bookshelf_clone_base_center, child bookshelf_clone_floor_2_piece, origin xyz=0.0 0.0 0.81 rpy=0 0 0
- added joint bookshelf_clone_left_side_piece_joint: type fixed, parent bookshelf_clone_origin, child bookshelf_clone_left_side_piece, origin xyz=0.2 0.88 0.45 rpy=0 0 0
- added joint bookshelf_clone_origin_joint: type fixed, parent room_link, child bookshelf_clone_origin, origin xyz=5.79168 4.55429 0 rpy=0 0 1.5707963
- added joint bookshelf_clone_right_side_piece_joint: type fixed, parent bookshelf_clone_origin, child bookshelf_clone_right_side_piece, origin xyz=0.2 0.0 0.45 rpy=0 0 0

Commit message: added tests for assignplaces, beliefstate, pickup, surfaces and urdf

File: knowledge/urdf/gz_sim_v1_openable_door.urdf (robot description, URDF)
Before this commit: robot hsrb_lab, 36 links, 35 joints
Links:
- added link base_footprint
Joints:
- added joint base_footprint_joint: type fixed, parent world, child base_footprint, origin xyz=0.5151 -0.506436 0 rpy=0 0 0
