Commit message: adapted rooms to new urdf naming convention

File: knowledge/urdf/suturo_rooms.urdf (robot description, URDF)
Before this commit: robot suturo_rooms, 63 links, 62 joints
Links:
- removed link door_hall_livingroom_1_door_center
- removed link door_hall_livingroom_1_door_handle_inside
- removed link door_hall_livingroom_1_door_handle_outside
- removed link door_hall_livingroom_1_door_hinge
- removed link door_hall_sleepingroom_1_door_center
- removed link door_hall_sleepingroom_1_door_handle_inside
- removed link door_hall_sleepingroom_1_door_handle_outside
- removed link door_hall_sleepingroom_1_door_hinge
- removed link door_livingroom_sleepingroom_1_door_center
- removed link door_livingroom_sleepingroom_1_door_handle_inside
- removed link door_livingroom_sleepingroom_1_door_handle_outside
- removed link door_livingroom_sleepingroom_1_door_hinge
- removed link livingroom_room_center_link
- removed link livingroom_room_corner_0_link
- removed link livingroom_room_corner_1_link
- removed link livingroom_room_corner_2_link
- removed link livingroom_room_corner_3_link
- removed link livingroom_room_corner_4_link
- removed link livingroom_room_corner_5_link
- removed link sleepingroom_room_center_link
- removed link sleepingroom_room_corner_0_link
- removed link sleepingroom_room_corner_1_link
- removed link sleepingroom_room_corner_2_link
- removed link sleepingroom_room_corner_3_link
- added link door_hall_living-room_1_door_center; collision box size=1.0 0.055 2; visual box size=1.0 0.055 2
- added link door_hall_living-room_1_door_handle_inside; collision box size=0.15 0.025 0.015; visual box size=0.15 0.025 0.015
- added link door_hall_living-room_1_door_handle_outside; collision box size=0.15 0.025 0.015; visual box size=0.15 0.025 0.015
- added link door_hall_living-room_1_door_hinge; collision box size=0.05 0.05 2; visual box size=0.05 0.05 2
- added link door_hall_sleeping-room_1_door_center; collision box size=1.0 0.055 2; visual box size=1.0 0.055 2
- added link door_hall_sleeping-room_1_door_handle_inside; collision box size=0.15 0.025 0.015; visual box size=0.15 0.025 0.015
- added link door_hall_sleeping-room_1_door_handle_outside; collision box size=0.15 0.025 0.015; visual box size=0.15 0.025 0.015
- added link door_hall_sleeping-room_1_door_hinge; collision box size=0.05 0.05 2; visual box size=0.05 0.05 2
- added link door_living-room_sleeping-room_1_door_center; collision box size=1.0 0.055 2; visual box size=1.0 0.055 2
- added link door_living-room_sleeping-room_1_door_handle_inside; collision box size=0.15 0.025 0.015; visual box size=0.15 0.025 0.015
- added link door_living-room_sleeping-room_1_door_handle_outside; collision box size=0.15 0.025 0.015; visual box size=0.15 0.025 0.015
- added link door_living-room_sleeping-room_1_door_hinge; collision box size=0.05 0.05 2; visual box size=0.05 0.05 2
- added link living-room_room_center_link; visual cylinder length=0 radius=0
- added link living-room_room_corner_0_link
- added link living-room_room_corner_1_link
- added link living-room_room_corner_2_link
- added link living-room_room_corner_3_link
- added link living-room_room_corner_4_link
- added link living-room_room_corner_5_link
- added link sleeping-room_room_center_link; visual cylinder length=0 radius=0
- added link sleeping-room_room_corner_0_link
- added link sleeping-room_room_corner_1_link
- added link sleeping-room_room_corner_2_link
- added link sleeping-room_room_corner_3_link
Joints:
- removed joint door_hall_livingroom_1_door_handle_inside_joint
- removed joint door_hall_livingroom_1_door_handle_outside_joint
- removed joint door_hall_livingroom_1_door_hinge_joint
- removed joint door_hall_livingroom_1_door_origin_revolute_joint
- removed joint door_hall_sleepingroom_1_door_handle_inside_joint
- removed joint door_hall_sleepingroom_1_door_handle_outside_joint
- removed joint door_hall_sleepingroom_1_door_hinge_joint
- removed joint door_hall_sleepingroom_1_door_origin_revolute_joint
- removed joint door_livingroom_sleepingroom_1_door_handle_inside_joint
- removed joint door_livingroom_sleepingroom_1_door_handle_outside_joint
- removed joint door_livingroom_sleepingroom_1_door_hinge_joint
- removed joint door_livingroom_sleepingroom_1_door_origin_revolute_joint
- removed joint livingroom_room_joint_0
- removed joint livingroom_room_joint_1
- removed joint livingroom_room_joint_2
- removed joint livingroom_room_joint_3
- removed joint livingroom_room_joint_4
- removed joint livingroom_room_joint_5
- removed joint sleepingroom_room_joint_0
- removed joint sleepingroom_room_joint_1
- removed joint sleepingroom_room_joint_2
- removed joint sleepingroom_room_joint_3
- removed joint world_livingroom_room_joint
- removed joint world_sleepingroom_room_joint
- added joint door_hall_living-room_1_door_handle_inside_joint: type fixed, parent door_hall_living-room_1_door_center, child door_hall_living-room_1_door_handle_inside, origin xyz=0.9 -0.06875 -0.13 rpy=0 0 0, axis 0 0 0, limit lower=0 upper=1.5708 effort=1 velocity=1
- added joint door_hall_living-room_1_door_handle_outside_joint: type fixed, parent door_hall_living-room_1_door_center, child door_hall_living-room_1_door_handle_outside, origin xyz=0.9 0.055 -0.13 rpy=0 0 0, axis 0 0 0, limit lower=0 upper=1.5708 effort=1 velocity=1
- added joint door_hall_living-room_1_door_hinge_joint: type fixed, parent urdf_offset, child door_hall_living-room_1_door_hinge, origin xyz=-2 3.5 1.045 rpy=0 0 0, axis 0 0 0, limit lower=0 upper=1.5708 effort=1 velocity=1
- added joint door_hall_living-room_1_door_origin_revolute_joint: type revolute, parent door_hall_living-room_1_door_hinge, child door_hall_living-room_1_door_center, origin xyz=0 0 0 rpy=0 0 1.57079632679, axis 0 0 1, limit lower=0 upper=1.5708 effort=100 velocity=10
- added joint door_hall_sleeping-room_1_door_handle_inside_joint: type fixed, parent door_hall_sleeping-room_1_door_center, child door_hall_sleeping-room_1_door_handle_inside, origin xyz=0.9 -0.06875 -0.13 rpy=0 0 0, axis 0 0 0, limit lower=0 upper=1.5708 effort=1 velocity=1
- added joint door_hall_sleeping-room_1_door_handle_outside_joint: type fixed, parent door_hall_sleeping-room_1_door_center, child door_hall_sleeping-room_1_door_handle_outside, origin xyz=0.9 0.055 -0.13 rpy=0 0 0, axis 0 0 0, limit lower=0 upper=1.5708 effort=1 velocity=1
- added joint door_hall_sleeping-room_1_door_hinge_joint: type fixed, parent urdf_offset, child door_hall_sleeping-room_1_door_hinge, origin xyz=-3 1.0 1.045 rpy=0 0 0, axis 0 0 0, limit lower=0 upper=1.5708 effort=1 velocity=1
- added joint door_hall_sleeping-room_1_door_origin_revolute_joint: type revolute, parent door_hall_sleeping-room_1_door_hinge, child door_hall_sleeping-room_1_door_center, origin xyz=0 0 0 rpy=0 0 1.57079632679, axis 0 0 1, limit lower=0 upper=1.5708 effort=100 velocity=10
- added joint door_living-room_sleeping-room_1_door_handle_inside_joint: type fixed, parent door_living-room_sleeping-room_1_door_center, child door_living-room_sleeping-room_1_door_handle_inside, origin xyz=0.9 -0.06875 -0.13 rpy=0 0 0, axis 0 0 0, limit lower=0 upper=1.5708 effort=1 velocity=1
- added joint door_living-room_sleeping-room_1_door_handle_outside_joint: type fixed, parent door_living-room_sleeping-room_1_door_center, child door_living-room_sleeping-room_1_door_handle_outside, origin xyz=0.9 0.055 -0.13 rpy=0 0 0, axis 0 0 0, limit lower=0 upper=1.5708 effort=1 velocity=1
- added joint door_living-room_sleeping-room_1_door_hinge_joint: type fixed, parent urdf_offset, child door_living-room_sleeping-room_1_door_hinge, origin xyz=-1.5 3 1.045 rpy=0 0 0, axis 0 0 0, limit lower=0 upper=1.5708 effort=1 velocity=1
- added joint door_living-room_sleeping-room_1_door_origin_revolute_joint: type revolute, parent door_living-room_sleeping-room_1_door_hinge, child door_living-room_sleeping-room_1_door_center, origin xyz=0 0 0 rpy=0 0 0, axis 0 0 1, limit lower=0 upper=1.5708 effort=100 velocity=10
- added joint living-room_room_joint_0: type fixed, parent living-room_room_center_link, child living-room_room_corner_0_link, origin xyz=-1.5 -3 0  rpy=0 0 0
- added joint living-room_room_joint_1: type fixed, parent living-room_room_center_link, child living-room_room_corner_1_link, origin xyz=1.5 -3 0  rpy=0 0 0
- added joint living-room_room_joint_2: type fixed, parent living-room_room_center_link, child living-room_room_corner_2_link, origin xyz=1.5 2 0  rpy=0 0 0
- added joint living-room_room_joint_3: type fixed, parent living-room_room_center_link, child living-room_room_corner_3_link, origin xyz=-3.5 2 0  rpy=0 0 0
- added joint living-room_room_joint_4: type fixed, parent living-room_room_center_link, child living-room_room_corner_4_link, origin xyz=-3.5 0 0  rpy=0 0 0
- added joint living-room_room_joint_5: type fixed, parent living-room_room_center_link, child living-room_room_corner_5_link, origin xyz=-1.5 0 0  rpy=0 0 0
- added joint sleeping-room_room_joint_0: type fixed, parent sleeping-room_room_center_link, child sleeping-room_room_corner_0_link, origin xyz=-1.5 -1.5 0  rpy=0 0 0
- added joint sleeping-room_room_joint_1: type fixed, parent sleeping-room_room_center_link, child sleeping-room_room_corner_1_link, origin xyz=1.5 -1.5 0  rpy=0 0 0
- added joint sleeping-room_room_joint_2: type fixed, parent sleeping-room_room_center_link, child sleeping-room_room_corner_2_link, origin xyz=1.5 1.5 0  rpy=0 0 0
- added joint sleeping-room_room_joint_3: type fixed, parent sleeping-room_room_center_link, child sleeping-room_room_corner_3_link, origin xyz=-1.5 1.5 0  rpy=0 0 0
- added joint world_living-room_room_joint: type fixed, parent urdf_offset, child living-room_room_center_link, origin xyz=1.5 3 0  rpy=0 0 0
- added joint world_sleeping-room_room_joint: type fixed, parent urdf_offset, child sleeping-room_room_center_link, origin xyz=-1.5 1.5 0  rpy=0 0 0

Commit message: added location calculation and verification

File: knowledge/urdf/suturo_rooms.urdf (robot description, URDF)
Before this commit: robot suturo_rooms, 63 links, 62 joints
Joints:
- joint base_footprint_joint: origin xyz=-4.0 -4.0 0.0 rpy=0 0 0 -> xyz=-4.0 -3.0 0.0 rpy=0 0 0
